File: Electronic Trombone.kicad_sch (KiCad schematic)
At the start: 0 parts

Commit message: completed oscillator schematic
Parts:
- added C1: 2.2n, symbol Device:C
- added C2: C, symbol Device:C
- added D1: 1N4148, Diode_THT:D_DO-35_SOD27_P7.62mm_Horizontal, symbol Diode:1N4148
- added J_In, J_Out: Screw_Terminal_01x01, symbol Connector:Screw_Terminal_01x01
- added Q1: NPN, symbol Simulation_SPICE:NPN
- added Q2: PNP, symbol Simulation_SPICE:PNP
- added R1, R_Fine: 1M, symbol Device:R_US
- added R2, R3, R4: R_US, symbol Device:R_US
- added RV1: R_Potentiometer_US, symbol Device:R_Potentiometer_US
- added RV_CoarseTuning, RV_FineTuning: 100k, symbol Device:R_Potentiometer_US
- added R_Coarse, R_In: 100k, symbol Device:R_US
- added R_CurrentLimit: 1k, symbol Device:R_US
- added TH_Coarse, TH_Fine, TH_In: 10k, symbol Device:Thermistor_US
- added U1: 40106, symbol 4xxx:40106
- added U2, U3: TL074, symbol Amplifier_Operational:TL074
Connections:
- new net: Q1.2 (B), Q2.1 (C), R1.2
- new net: RV_FineTuning.2, R_Fine.1
- new net: R_Fine.2, TH_Fine.1
- new net: R_In.2, TH_In.1
- new net: RV_CoarseTuning.2, R_Coarse.1
- new net: R_Coarse.2, TH_Coarse.1
- new net: R3.1, R4.2, U3.2 (-)
- new net: R3.2, RV1.3, U3.1
- new net: C1.1, D1.1 (K), Q1.1 (C), U1.1, U2.3 (+)
- new net: D1.2 (A), U1.2
- new net: C2.2, R2.1, U3.3 (+)
- new net: R_CurrentLimit.1, U2.1, U2.2 (-)
- new net +12V: R1.1
- new net -12V: RV_CoarseTuning.3, RV_FineTuning.3
- new net Amp In: C2.1, R_CurrentLimit.2
- new net Core In: Q2.2 (B), TH_Coarse.2, TH_Fine.2, TH_In.2
- new net GND: C1.2, Q1.3 (E), Q2.3 (E), R2.2, R4.1, RV1.1, RV_CoarseTuning.1, RV_FineTuning.1
- new net In: J_In.1 (Pin_1), R_In.1
- new net Out: J_Out.1 (Pin_1), RV1.2
