File: KiCad/Oscillator.kicad_sch (KiCad schematic)
At the start: 36 parts, among them Q1 NPN, Q2 PNP, Q3 NPN, Q4 PNP, U1 40106, U2 TL074

Commit message: finalizing schematic
Parts:
- R11: renamed from R13; value 100k -> R_US
- R15: renamed from R51; value 2.5k -> R_US
- R17: renamed from R8; value 1k -> R_US
- R18: renamed from R49; value 100k -> R_US
- R20: renamed from R50; value 100k -> R_US
- R24: renamed from R12; value 2.5k -> R_US
- R9: renamed from R5; value 100k -> R_US
- renumbered R1 to R10, R2 to R12, R3 to R13, R6 to R14, R7 to R16, R9 to R19, R10 to R21, R11 to R22, R14 to R23, RV2 to RV1, RV3 to RV2, RV5 to RV3, U1 to U2, U2 to U3
Other:
- note removed: "Replacable: a component (e.g. a resistor) should be through hole so that I can adjust its value when the PCB arrives"
