File: KiCad/Oscillator.kicad_sch (KiCad schematic)
At the start: 36 parts, among them Q1 NPN, Q2 PNP, Q3 NPN, Q4 PNP, U4 40106, U5 TL074

Commit message: started pcb layout
Connections:
- net Sch Inv In 1: now reaches C1.1, D1.1 (K), Q1.1 (C), U4.1, U5.3 (+)
- net Sch Inv In 2: now reaches C3.1, D2.1 (K), Q3.1 (C), U4.9, U5.5 (+)
- net Tuning 1: now reaches R17.1, RV9.2
- net Tuning 2: now reaches R26.1, RV11.2
Other:
- moved on the sheet: RV11, RV9
Changed lines of the file:
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@@
 	(wire
 		(pts
-			(xy 30.48 58.42) (xy 34.29 58.42)
+			(xy 21.59 58.42) (xy 25.4 58.42)
 		)
 		(stroke
@@
 	(wire
 		(pts
-			(xy 30.48 142.24) (xy 34.29 142.24)
+			(xy 21.59 142.24) (xy 25.4 142.24)
 		)
 		(stroke
@@
 	(wire
 		(pts
-			(xy 38.1 71.12) (xy 40.64 71.12)
+			(xy 29.21 71.12) (xy 40.64 71.12)
 		)
 		(stroke
@@
 	(wire
 		(pts
-			(xy 34.29 58.42) (xy 34.29 67.31)
+			(xy 25.4 58.42) (xy 25.4 67.31)
 		)
 		(stroke
@@
 	(wire
 		(pts
-			(xy 34.29 142.24) (xy 34.29 151.13)
+			(xy 25.4 142.24) (xy 25.4 151.13)
 		)
 		(stroke
@@
 	(wire
 		(pts
-			(xy 38.1 154.94) (xy 40.64 154.94)
+			(xy 29.21 154.94) (xy 40.64 154.94)
 		)
 		(stroke
@@
 		)
 	)
+	(label "Sch Inv In 1"
+		(at 118.11 53.34 0)
+		(effects
+			(font
+				(size 1.27 1.27)
+			)
+			(justify left bottom)
+		)
+	)
 	(label "Mix In 2"
 		(at 186.69 118.11 0)
@@
 		)
 	)
+	(label "Sch Inv In 2"
+		(at 118.11 130.81 0)
+		(effects
+			(font
+				(size 1.27 1.27)
+			)
+			(justify left bottom)
+		)
+	)
+	(label "Tuning 1"
+		(at 31.75 71.12 0)
+		(effects
+			(font
+				(size 1.27 1.27)
+			)
+			(justify left bottom)
+		)
+	)
 	(label "Sch Inv Out 1"
 		(at 156.21 46.99 0)
@@
 		)
 	)
+	(label "Tuning 2"
+		(at 31.75 154.94 0)
+		(effects
+			(font
+				(size 1.27 1.27)
+			)
+			(justify left bottom)
+		)
+	)
 	(label "Core In 1"
 		(at 85.09 64.77 0)
@@
 	(symbol
 		(lib_id "power:GND")
-		(at 30.48 142.24 0)
+		(at 21.59 142.24 0)
 		(unit 1)
 		(body_style 1)
@@
 		(fields_autoplaced yes)
 		(property "Reference" "#PWR041"
-			(at 30.48 148.59 0)
+			(at 21.59 148.59 0)
 			(hide yes)
 			(show_name no)
@@
 		)
 		(property "Value" "GND"
-			(at 30.48 147.32 0)
+			(at 21.59 147.32 0)
 			(show_name no)
 			(do_not_autoplace no)
@@
 		)
 		(property "Footprint" ""
-			(at 30.48 142.24 0)
+			(at 21.59 142.24 0)
 			(hide yes)
 			(show_name no)
@@
 		)
 		(property "Datasheet" ""
-			(at 30.48 142.24 0)
+			(at 21.59 142.24 0)
 			(hide yes)
 			(show_name no)
@@
 		)
 		(property "Description" "Power symbol creates a global label with name \"GND\" , ground"
-			(at 30.48 142.24 0)
+			(at 21.59 142.24 0)
 			(hide yes)
 			(show_name no)
@@
 	(symbol
 		(lib_id "power:-9V")
-		(at 34.29 158.75 180)
+		(at 25.4 158.75 180)
 		(unit 1)
 		(body_style 1)
@@
 		(fields_autoplaced yes)
 		(property "Reference" "#PWR043"
-			(at 34.29 154.94 0)
+			(at 25.4 154.94 0)
 			(hide yes)
 			(show_name no)
@@
 		)
 		(property "Value" "-9V"
-			(at 34.29 163.83 0)
+			(at 25.4 163.83 0)
 			(show_name no)
 			(do_not_autoplace no)
@@
 		)
 		(property "Footprint" ""
-			(at 34.29 158.75 0)
+			(at 25.4 158.75 0)
 			(hide yes)
 			(show_name no)
@@
 		)
 		(property "Datasheet" ""
-			(at 34.29 158.75 0)
+			(at 25.4 158.75 0)
 			(hide yes)
 			(show_name no)
@@
 		)
 		(property "Description" "Power symbol creates a global label with name \"-9V\""
-			(at 34.29 158.75 0)
+			(at 25.4 158.75 0)
 			(hide yes)
 			(show_name no)
@@
 	(symbol
 		(lib_id "Device:R_Potentiometer_US")
-		(at 34.29 154.94 0)
+		(at 25.4 154.94 0)
 		(unit 1)
 		(body_style 1)
@@
 		(fields_autoplaced yes)
 		(property "Reference" "RV11"
-			(at 31.75 153.6699 0)
+			(at 22.86 153.6699 0)
 			(show_name no)
 			(do_not_autoplace no)
@@
 		)
 		(property "Value" "100k"
-			(at 31.75 156.2099 0)
+			(at 22.86 156.2099 0)
 			(show_name no)
 			(do_not_autoplace no)
@@
 		)
 		(property "Footprint" "Potentiometer 100k PTV09A-2020F-B104:Potentiometer 100k PTV09A-2020F-B104"
-			(at 34.29 154.94 0)
+			(at 25.4 154.94 0)
 			(hide yes)
 			(show_name no)
@@
 		)
 		(property "Datasheet" ""
-			(at 34.29 154.94 0)
+			(at 25.4 154.94 0)
 			(hide yes)
 			(show_name no)
@@
 		)
 		(property "Description" "Potentiometer, US symbol"
-			(at 34.29 154.94 0)
+			(at 25.4 154.94 0)
 			(hide yes)
 			(show_name no)
@@
 		)
 		(property "Sim.Device" "R"
-			(at 34.29 154.94 0)
+			(at 25.4 154.94 0)
 			(hide yes)
 			(show_name no)
@@
 		)
 		(property "Sim.Type" "POT"
-			(at 34.29 154.94 0)
+			(at 25.4 154.94 0)
 			(hide yes)
 			(show_name no)
@@
 		)
 		(property "Sim.Pins" "1=r0 2=wiper 3=r1"
-			(at 34.29 154.94 0)
+			(at 25.4 154.94 0)
 			(hide yes)
 			(show_name no)
@@
 	(symbol
 		(lib_id "Device:R_Potentiometer_US")
-		(at 34.29 71.12 0)
+		(at 25.4 71.12 0)
 		(unit 1)
 		(body_style 1)
@@
 		(fields_autoplaced yes)
 		(property "Reference" "RV9"
-			(at 31.75 69.8499 0)
+			(at 22.86 69.8499 0)
 			(show_name no)
 			(do_not_autoplace no)
@@
 		)
 		(property "Value" "100k"
-			(at 31.75 72.3899 0)
+			(at 22.86 72.3899 0)
 			(show_name no)
 			(do_not_autoplace no)
@@
 		)
 		(property "Footprint" "Potentiometer 100k PTV09A-2020F-B104:Potentiometer 100k PTV09A-2020F-B104"
-			(at 34.29 71.12 0)
+			(at 25.4 71.12 0)
 			(hide yes)
 			(show_name no)
@@
 		)
 		(property "Datasheet" ""
-			(at 34.29 71.12 0)
+			(at 25.4 71.12 0)
 			(hide yes)
 			(show_name no)
@@
 		)
 		(property "Description" "Potentiometer, US symbol"
-			(at 34.29 71.12 0)
+			(at 25.4 71.12 0)
 			(hide yes)
 			(show_name no)
@@
 		)
 		(property "Sim.Device" "R"
-			(at 34.29 71.12 0)
+			(at 25.4 71.12 0)
 			(hide yes)
 			(show_name no)
@@
 		)
 		(property "Sim.Type" "POT"
-			(at 34.29 71.12 0)
+			(at 25.4 71.12 0)
 			(hide yes)
 			(show_name no)
@@
 		)
 		(property "Sim.Pins" "1=r0 2=wiper 3=r1"
-			(at 34.29 71.12 0)
+			(at 25.4 71.12 0)
 			(hide yes)
 			(show_name no)
@@
 	(symbol
 		(lib_id "power:GND")
-		(at 30.48 58.42 0)
+		(at 21.59 58.42 0)
 		(unit 1)
 		(body_style 1)
@@
 		(fields_autoplaced yes)
 		(property "Reference" "#PWR029"
-			(at 30.48 64.77 0)
+			(at 21.59 64.77 0)
 			(hide yes)
 			(show_name no)
@@
 		)
 		(property "Value" "GND"
-			(at 30.48 63.5 0)
+			(at 21.59 63.5 0)
 			(show_name no)
 			(do_not_autoplace no)
@@
 		)
 		(property "Footprint" ""
-			(at 30.48 58.42 0)
+			(at 21.59 58.42 0)
 			(hide yes)
 			(show_name no)
@@
 		)
 		(property "Datasheet" ""
-			(at 30.48 58.42 0)
+			(at 21.59 58.42 0)
 			(hide yes)
 			(show_name no)
@@
 		)
 		(property "Description" "Power symbol creates a global label with name \"GND\" , ground"
-			(at 30.48 58.42 0)
+			(at 21.59 58.42 0)
 			(hide yes)
 			(show_name no)
@@
 	(symbol
 		(lib_id "power:-9V")
-		(at 34.29 74.93 180)
+		(at 25.4 74.93 180)
 		(unit 1)
 		(body_style 1)
@@
 		(fields_autoplaced yes)
 		(property "Reference" "#PWR033"
-			(at 34.29 71.12 0)
+			(at 25.4 71.12 0)
 			(hide yes)
 			(show_name no)
@@
 		)
 		(property "Value" "-9V"
-			(at 34.29 80.01 0)
+			(at 25.4 80.01 0)
 			(show_name no)
 			(do_not_autoplace no)
@@
 		)
 		(property "Footprint" ""
-			(at 34.29 74.93 0)
+			(at 25.4 74.93 0)
 			(hide yes)
 			(show_name no)
@@
 		)
 		(property "Datasheet" ""
-			(at 34.29 74.93 0)
+			(at 25.4 74.93 0)
 			(hide yes)
 			(show_name no)
@@
 		)
 		(property "Description" "Power symbol creates a global label with name \"-9V\""
-			(at 34.29 74.93 0)
+			(at 25.4 74.93 0)
 			(hide yes)
 			(show_name no)

Commit message: added osc core and tuning to pcb layout
Parts:
- R19, R28: value 2.5k -> 2.4k; footprint Resistor_SMD:R_0603_1608Metric -> Resistor_SMD:R_0201_0603Metric
Connections:
- net Mix In 1: now also U5.6 (-), U5.7; no longer U5.1, U5.2 (-)
- net Mix In 2: now also U5.1, U5.2 (-); no longer U5.6 (-), U5.7
- net Out: now also U5.13 (-), U5.14; no longer U5.8, U5.9 (-)
- net Sch Inv In 1: now also U5.5 (+); no longer U5.3 (+)
- net Sch Inv In 2: now also U5.3 (+); no longer U5.5 (+)
- net at R20.2, R21.2: now also U5.12 (+); no longer U5.10 (+)
Changed lines of the file:
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@@
 		(lib_id "Amplifier_Operational:TL074")
 		(at 149.86 72.39 0)
-		(unit 1)
+		(unit 2)
 		(body_style 1)
 		(exclude_from_sim no)
@@
 				(path "/931827f3-33b7-460f-8885-7db258da2648/c601a773-7a8a-4dbf-b4ab-ef5ea2e44138"
 					(reference "U5")
-					(unit 1)
+					(unit 2)
 				)
 			)
@@
 		(lib_id "Amplifier_Operational:TL074")
 		(at 149.86 149.86 0)
-		(unit 2)
+		(unit 1)
 		(body_style 1)
 		(exclude_from_sim no)
@@
 				(path "/931827f3-33b7-460f-8885-7db258da2648/c601a773-7a8a-4dbf-b4ab-ef5ea2e44138"
 					(reference "U5")
-					(unit 2)
+					(unit 1)
 				)
 			)
@@
 		(lib_id "Amplifier_Operational:TL074")
 		(at 234.95 110.49 0)
-		(unit 3)
+		(unit 4)
 		(body_style 1)
 		(exclude_from_sim no)
@@
 				(path "/931827f3-33b7-460f-8885-7db258da2648/c601a773-7a8a-4dbf-b4ab-ef5ea2e44138"
 					(reference "U5")
-					(unit 3)
+					(unit 4)
 				)
 			)
@@
 			)
 		)
-		(property "Value" "2.5k"
+		(property "Value" "2.4k"
 			(at 66.04 102.8699 0)
 			(show_name no)
@@
 			)
 		)
-		(property "Footprint" "Resistor_SMD:R_0603_1608Metric"
+		(property "Footprint" "Resistor_SMD:R_0201_0603Metric"
 			(at 64.516 101.854 90)
 			(hide yes)
@@
 			)
 		)
-		(property "Value" "2.5k"
+		(property "Value" "2.4k"
 			(at 66.04 186.6899 0)
 			(show_name no)
@@
 			)
 		)
-		(property "Footprint" "Resistor_SMD:R_0603_1608Metric"
+		(property "Footprint" "Resistor_SMD:R_0201_0603Metric"
 			(at 64.516 185.674 90)
 			(hide yes)

Commit message: routed oscillator
Parts:
- renumbered U5 to U7
Connections:
- net Mix In 1: now also RV10.3; no longer RV10.1
- net Mix In 2: now also RV10.1; no longer RV10.3
Changed lines of the file:
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@@
 		(in_pos_files yes)
 		(dnp no)
-		(property "Reference" "U5"
+		(property "Reference" "U7"
 			(at 234.95 100.33 0)
 			(show_name no)
@@
 			(project "Electronic Trombone"
 				(path "/931827f3-33b7-460f-8885-7db258da2648/c601a773-7a8a-4dbf-b4ab-ef5ea2e44138"
-					(reference "U5")
+					(reference "U7")
 					(unit 4)
 				)
@@
 		(lib_id "Device:R_Potentiometer_US")
 		(at 195.58 107.95 0)
+		(mirror x)
 		(unit 1)
 		(body_style 1)
@@
 		(in_pos_files yes)
 		(dnp no)
-		(fields_autoplaced yes)
 		(property "Reference" "RV10"
-			(at 193.04 106.6799 0)
+			(at 193.04 109.2201 0)
 			(show_name no)
 			(do_not_autoplace no)
@@
 		)
 		(property "Value" "100k"
-			(at 193.04 109.2199 0)
-			(show_name no)
-			(do_not_autoplace no)
+			(at 193.04 106.6801 0)
+			(show_name no)
+			(do_not_autoplace no)

Commit message: started filter layout
Connections:
- net Out: now also U7.1, U7.2 (-); no longer U7.13 (-), U7.14
- net at R20.2, R21.2: now also U7.3 (+); no longer U7.12 (+)
Changed lines of the file:
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@@
 		(lib_id "Amplifier_Operational:TL074")
 		(at 234.95 110.49 0)
-		(unit 4)
+		(unit 1)
 		(body_style 1)
 		(exclude_from_sim no)
@@
 				(path "/931827f3-33b7-460f-8885-7db258da2648/c601a773-7a8a-4dbf-b4ab-ef5ea2e44138"
 					(reference "U7")
-					(unit 4)
+					(unit 1)
 				)
 			)
