File: KiCad/buttons.kicad_sch (KiCad schematic)
At the start: 8 parts, among them J3 691137710003, J4 691137710002, SW1 SW_Push, SW2 SW_Push, SW3 SW_Push

Commit message: added push button footprints
Parts:
- SW1, SW2, SW3: footprint (none) -> Switch Push Button D6R90F2LFS:D6R90_CNK
Changed lines of the file:
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@@
 			)
 		)
-		(property "Footprint" ""
+		(property "Footprint" "Switch Push Button D6R90F2LFS:D6R90_CNK"
 			(at 34.29 82.55 0)
 			(hide yes)
@@
 			)
 		)
-		(property "Footprint" ""
+		(property "Footprint" "Switch Push Button D6R90F2LFS:D6R90_CNK"
 			(at 34.29 54.61 0)
 			(hide yes)
@@
 			)
 		)
-		(property "Footprint" ""
+		(property "Footprint" "Switch Push Button D6R90F2LFS:D6R90_CNK"
 			(at 34.29 68.58 0)
 			(hide yes)
