File: KiCad/Envelope Generator.kicad_sch (KiCad schematic)
At the start: 36 parts, among them U10 TL074, U9 TL074

Commit message: added power switch, decoupling caps, and unused IC pins
Parts:
- renumbered R54 to R50, R55 to R51, R56 to R52, R57 to R53, R58 to R54, R59 to R55, R60 to R56, R61 to R57, R62 to R58, R63 to R59, R64 to R60, R65 to R61, R66 to R62, R67 to R63, R68 to R64, R69 to R65, R70 to R66, R71 to R67
Changed lines of the file:
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@@
 		(dnp no)
 		(fields_autoplaced yes)
-		(property "Reference" "R71"
+		(property "Reference" "R67"
 			(at 143.51 152.4 90)
 			(show_name no)
@@
 			(project "Electronic Trombone"
 				(path "/931827f3-33b7-460f-8885-7db258da2648/77fe3443-32fb-46cd-8502-6f8d1ae6ff63"
-					(reference "R71")
+					(reference "R67")
 					(unit 1)
 				)
@@
 		(dnp no)
 		(fields_autoplaced yes)
-		(property "Reference" "#PWR074"
+		(property "Reference" "#PWR065"
 			(at 49.53 162.56 0)
 			(hide yes)
@@
 			(project "Electronic Trombone"
 				(path "/931827f3-33b7-460f-8885-7db258da2648/77fe3443-32fb-46cd-8502-6f8d1ae6ff63"
-					(reference "#PWR074")
+					(reference "#PWR065")
 					(unit 1)
 				)
@@
 		(dnp no)
 		(fields_autoplaced yes)
-		(property "Reference" "R70"
+		(property "Reference" "R66"
 			(at 184.15 147.32 90)
 			(show_name no)
@@
 			(project "Electronic Trombone"
 				(path "/931827f3-33b7-460f-8885-7db258da2648/77fe3443-32fb-46cd-8502-6f8d1ae6ff63"
-					(reference "R70")
+					(reference "R66")
 					(unit 1)
 				)
@@
 		(dnp no)
 		(fields_autoplaced yes)
-		(property "Reference" "R56"
+		(property "Reference" "R52"
 			(at 168.91 34.29 90)
 			(show_name no)
@@
 			(project "Electronic Trombone"
 				(path "/931827f3-33b7-460f-8885-7db258da2648/77fe3443-32fb-46cd-8502-6f8d1ae6ff63"
-					(reference "R56")
+					(reference "R52")
 					(unit 1)
 				)
@@
 		(dnp no)
 		(fields_autoplaced yes)
-		(property "Reference" "R60"
+		(property "Reference" "R56"
 			(at 143.51 81.28 90)
 			(show_name no)
@@
 			(project "Electronic Trombone"
 				(path "/931827f3-33b7-460f-8885-7db258da2648/77fe3443-32fb-46cd-8502-6f8d1ae6ff63"
-					(reference "R60")
+					(reference "R56")
 					(unit 1)
 				)
@@
 		(dnp no)
 		(fields_autoplaced yes)
-		(property "Reference" "R55"
+		(property "Reference" "R51"
 			(at 114.3 34.29 90)
 			(show_name no)
@@
 			(project "Electronic Trombone"
 				(path "/931827f3-33b7-460f-8885-7db258da2648/77fe3443-32fb-46cd-8502-6f8d1ae6ff63"
-					(reference "R55")
+					(reference "R51")
 					(unit 1)
 				)
@@
 		(dnp no)
 		(fields_autoplaced yes)
-		(property "Reference" "R62"
+		(property "Reference" "R58"
 			(at 52.07 95.2499 0)
 			(show_name no)
@@
 			(project "Electronic Trombone"
 				(path "/931827f3-33b7-460f-8885-7db258da2648/77fe3443-32fb-46cd-8502-6f8d1ae6ff63"
-					(reference "R62")
+					(reference "R58")
 					(unit 1)
 				)
@@
 		(dnp no)
 		(fields_autoplaced yes)
-		(property "Reference" "#PWR068"
+		(property "Reference" "#PWR059"
 			(at 184.15 46.99 0)
 			(hide yes)
@@
 			(project "Electronic Trombone"
 				(path "/931827f3-33b7-460f-8885-7db258da2648/77fe3443-32fb-46cd-8502-6f8d1ae6ff63"
-					(reference "#PWR068")
+					(reference "#PWR059")
 					(unit 1)
 				)
@@
 		(dnp no)
 		(fields_autoplaced yes)
-		(property "Reference" "R69"
+		(property "Reference" "R65"
 			(at 91.44 151.1299 0)
 			(show_name no)
@@
 			(project "Electronic Trombone"
 				(path "/931827f3-33b7-460f-8885-7db258da2648/77fe3443-32fb-46cd-8502-6f8d1ae6ff63"
-					(reference "R69")
+					(reference "R65")
 					(unit 1)
 				)
@@
 		(dnp no)
 		(fields_autoplaced yes)
-		(property "Reference" "#PWR069"
+		(property "Reference" "#PWR060"
 			(at 31.75 48.26 0)
 			(hide yes)
@@
 			(project "Electronic Trombone"
 				(path "/931827f3-33b7-460f-8885-7db258da2648/77fe3443-32fb-46cd-8502-6f8d1ae6ff63"
-					(reference "#PWR069")
+					(reference "#PWR060")
 					(unit 1)
 				)
@@
 		(dnp no)
 		(fields_autoplaced yes)
-		(property "Reference" "R59"
+		(property "Reference" "R55"
 			(at 48.26 35.56 90)
 			(show_name no)
@@
 			(project "Electronic Trombone"
 				(path "/931827f3-33b7-460f-8885-7db258da2648/77fe3443-32fb-46cd-8502-6f8d1ae6ff63"
-					(reference "R59")
+					(reference "R55")
 					(unit 1)
 				)
@@
 		(dnp no)
 		(fields_autoplaced yes)
-		(property "Reference" "R61"
+		(property "Reference" "R57"
 			(at 36.83 95.2499 0)
 			(show_name no)
@@
 			(project "Electronic Trombone"
 				(path "/931827f3-33b7-460f-8885-7db258da2648/77fe3443-32fb-46cd-8502-6f8d1ae6ff63"
-					(reference "R61")
+					(reference "R57")
 					(unit 1)
 				)
@@
 		(dnp no)
 		(fields_autoplaced yes)
-		(property "Reference" "R68"
+		(property "Reference" "R64"
 			(at 52.07 151.1299 0)
 			(show_name no)
@@
 			(project "Electronic Trombone"
 				(path "/931827f3-33b7-460f-8885-7db258da2648/77fe3443-32fb-46cd-8502-6f8d1ae6ff63"
-					(reference "R68")
+					(reference "R64")
 					(unit 1)
 				)
@@
 		(dnp no)
 		(fields_autoplaced yes)
-		(property "Reference" "R58"
+		(property "Reference" "R54"
 			(at 38.1 35.56 90)
 			(show_name no)
@@
 			(project "Electronic Trombone"
 				(path "/931827f3-33b7-460f-8885-7db258da2648/77fe3443-32fb-46cd-8502-6f8d1ae6ff63"
-					(reference "R58")
+					(reference "R54")
 					(unit 1)
 				)
@@
 		(dnp no)
 		(fields_autoplaced yes)
-		(property "Reference" "R57"
+		(property "Reference" "R53"
 			(at 176.53 34.29 90)
 			(show_name no)
@@
 			(project "Electronic Trombone"
 				(path "/931827f3-33b7-460f-8885-7db258da2648/77fe3443-32fb-46cd-8502-6f8d1ae6ff63"
-					(reference "R57")
+					(reference "R53")
 					(unit 1)
 				)
@@
 		(dnp no)
 		(fields_autoplaced yes)
-		(property "Reference" "#PWR070"
+		(property "Reference" "#PWR061"
 			(at 54.61 38.1 0)
 			(hide yes)
@@
 			(project "Electronic Trombone"
 				(path "/931827f3-33b7-460f-8885-7db258da2648/77fe3443-32fb-46cd-8502-6f8d1ae6ff63"
-					(reference "#PWR070")
+					(reference "#PWR061")
 					(unit 1)
 				)
@@
 		(dnp no)
 		(fields_autoplaced yes)
-		(property "Reference" "R66"
+		(property "Reference" "R62"
 			(at 143.51 137.16 90)
 			(show_name no)
@@
 			(project "Electronic Trombone"
 				(path "/931827f3-33b7-460f-8885-7db258da2648/77fe3443-32fb-46cd-8502-6f8d1ae6ff63"
-					(reference "R66")
+					(reference "R62")
 					(unit 1)
 				)
@@
 		(dnp no)
 		(fields_autoplaced yes)
-		(property "Reference" "#PWR067"
+		(property "Reference" "#PWR058"
 			(at 121.92 46.99 0)
 			(hide yes)
@@
 			(project "Electronic Trombone"
 				(path "/931827f3-33b7-460f-8885-7db258da2648/77fe3443-32fb-46cd-8502-6f8d1ae6ff63"
-					(reference "#PWR067")
+					(reference "#PWR058")
 					(unit 1)
 				)
@@
 		(dnp no)
 		(fields_autoplaced yes)
-		(property "Reference" "#PWR076"
+		(property "Reference" "#PWR067"
 			(at 34.29 175.26 0)
 			(hide yes)
@@
 			(project "Electronic Trombone"
 				(path "/931827f3-33b7-460f-8885-7db258da2648/77fe3443-32fb-46cd-8502-6f8d1ae6ff63"
-					(reference "#PWR076")
+					(reference "#PWR067")
 					(unit 1)
 				)
@@
 		(dnp no)
 		(fields_autoplaced yes)
-		(property "Reference" "#PWR073"
+		(property "Reference" "#PWR064"
 			(at 34.29 119.38 0)
 			(hide yes)
@@
 			(project "Electronic Trombone"
 				(path "/931827f3-33b7-460f-8885-7db258da2648/77fe3443-32fb-46cd-8502-6f8d1ae6ff63"
-					(reference "#PWR073")
+					(reference "#PWR064")
 					(unit 1)
 				)
@@
 		(dnp no)
 		(fields_autoplaced yes)
-		(property "Reference" "R63"
+		(property "Reference" "R59"
 			(at 91.44 95.2499 0)
 			(show_name no)
@@
 			(project "Electronic Trombone"
 				(path "/931827f3-33b7-460f-8885-7db258da2648/77fe3443-32fb-46cd-8502-6f8d1ae6ff63"
-					(reference "R63")
+					(reference "R59")
 					(unit 1)
 				)
@@
 		(dnp no)
 		(fields_autoplaced yes)
-		(property "Reference" "R54"
+		(property "Reference" "R50"
 			(at 106.68 34.29 90)
 			(show_name no)
@@
 			(project "Electronic Trombone"
 				(path "/931827f3-33b7-460f-8885-7db258da2648/77fe3443-32fb-46cd-8502-6f8d1ae6ff63"
-					(reference "R54")
+					(reference "R50")
 					(unit 1)
 				)
@@
 		(dnp no)
 		(fields_autoplaced yes)
-		(property "Reference" "#PWR075"
+		(property "Reference" "#PWR066"
 			(at 156.21 167.64 0)
 			(hide yes)
@@
 			(project "Electronic Trombone"
 				(path "/931827f3-33b7-460f-8885-7db258da2648/77fe3443-32fb-46cd-8502-6f8d1ae6ff63"
-					(reference "#PWR075")
+					(reference "#PWR066")
 					(unit 1)
 				)
@@
 		(dnp no)
 		(fields_autoplaced yes)
-		(property "Reference" "#PWR071"
+		(property "Reference" "#PWR062"
 			(at 49.53 106.68 0)
 			(hide yes)
@@
 			(project "Electronic Trombone"
 				(path "/931827f3-33b7-460f-8885-7db258da2648/77fe3443-32fb-46cd-8502-6f8d1ae6ff63"
-					(reference "#PWR071")
+					(reference "#PWR062")
 					(unit 1)
 				)
@@
 		(dnp no)
 		(fields_autoplaced yes)
-		(property "Reference" "R65"
+		(property "Reference" "R61"
 			(at 143.51 96.52 90)
 			(show_name no)
@@
 			(project "Electronic Trombone"
 				(path "/931827f3-33b7-460f-8885-7db258da2648/77fe3443-32fb-46cd-8502-6f8d1ae6ff63"
-					(reference "R65")
+					(reference "R61")
 					(unit 1)
 				)
@@
 		(dnp no)
 		(fields_autoplaced yes)
-		(property "Reference" "R64"
+		(property "Reference" "R60"
 			(at 184.15 91.44 90)
 			(show_name no)
@@
 			(project "Electronic Trombone"
 				(path "/931827f3-33b7-460f-8885-7db258da2648/77fe3443-32fb-46cd-8502-6f8d1ae6ff63"
-					(reference "R64")
+					(reference "R60")
 					(unit 1)
 				)
@@
 		(dnp no)
 		(fields_autoplaced yes)
-		(property "Reference" "#PWR072"
+		(property "Reference" "#PWR063"
 			(at 156.21 111.76 0)
 			(hide yes)
@@
 			(project "Electronic Trombone"
 				(path "/931827f3-33b7-460f-8885-7db258da2648/77fe3443-32fb-46cd-8502-6f8d1ae6ff63"
-					(reference "#PWR072")
+					(reference "#PWR063")
 					(unit 1)
 				)
@@
 		(dnp no)
 		(fields_autoplaced yes)
-		(property "Reference" "R67"
+		(property "Reference" "R63"
 			(at 36.83 151.1299 0)
 			(show_name no)
@@
 			(project "Electronic Trombone"
 				(path "/931827f3-33b7-460f-8885-7db258da2648/77fe3443-32fb-46cd-8502-6f8d1ae6ff63"
-					(reference "R67")
+					(reference "R63")
 					(unit 1)
 				)
