File: KiCad/Filter.kicad_sch (KiCad schematic)
At the start: 25 parts, among them U7 TL074, U8 TL074

Commit message: started filter layout
Parts:
- renumbered D6 to D5, D9 to D6, D5 to D7, D7 to D8, D8 to D9
Connections:
- net Processed Control: now also U7.6 (-), U7.7; no longer U7.1, U7.2 (-)
- net at D7.2 (A), R41.1, R43.2: now also U7.5 (+); no longer U7.3 (+)
- net at R37.1, R38.2: now also U7.13 (-); no longer U7.6 (-)
- net Signal In w. +Offset: now reaches D3.2 (A), R37.2, R39.1
- net at R40.1, R42.2: now also U7.12 (+); no longer U7.5 (+)
- net Signal In w. -Offset: now reaches D6.1 (K), R44.2, R46.1
- net at R39.2: now also U7.14; no longer U7.7
Other:
- note removed: "Signal In with neg. offset"
- note removed: "Signal In with pos. offset"
Changed lines of the file:
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@@
 		)
 	)
-	(text "Signal In with neg. offset"
-		(exclude_from_sim no)
-		(at 235.458 102.616 0)
-		(effects
-			(font
-				(size 1.27 1.27)
-			)
-		)
-	)
 	(text "100mV pp., centered at 0V"
 		(exclude_from_sim no)
@@
 		)
 	)
-	(text "Signal In with pos. offset"
-		(exclude_from_sim no)
-		(at 235.458 51.816 0)
-		(effects
-			(font
-				(size 1.27 1.27)
-			)
-		)
-	)
 	(junction
 		(at 68.58 74.93)
@@
 		)
 	)
+	(label "Signal In w. -Offset"
+		(at 247.65 100.33 180)
+		(effects
+			(font
+				(size 1.27 1.27)
+			)
+			(justify right bottom)
+		)
+	)
+	(label "Signal In w. +Offset"
+		(at 247.65 53.34 180)
+		(effects
+			(font
+				(size 1.27 1.27)
+			)
+			(justify right bottom)
+		)
+	)
 	(hierarchical_label "Signal In"
 		(shape input)
@@
 		(dnp no)
 		(fields_autoplaced yes)
-		(property "Reference" "D7"
+		(property "Reference" "D8"
 			(at 71.12 85.0899 90)
 			(show_name no)
@@
 			(project "Electronic Trombone"
 				(path "/931827f3-33b7-460f-8885-7db258da2648/6d65ef8f-8235-46d4-95e7-69caf9b93e91"
-					(reference "D7")
+					(reference "D8")
 					(unit 1)
 				)
@@
 		(lib_id "Amplifier_Operational:TL074")
 		(at 92.71 77.47 0)
-		(unit 1)
+		(unit 2)
 		(body_style 1)
 		(exclude_from_sim no)
@@
 				(path "/931827f3-33b7-460f-8885-7db258da2648/6d65ef8f-8235-46d4-95e7-69caf9b93e91"
 					(reference "U7")
-					(unit 1)
+					(unit 2)
 				)
 			)
@@
 		(dnp no)
 		(fields_autoplaced yes)
-		(property "Reference" "D5"
+		(property "Reference" "D7"
 			(at 71.12 77.4699 90)
 			(show_name no)
@@
 			(project "Electronic Trombone"
 				(path "/931827f3-33b7-460f-8885-7db258da2648/6d65ef8f-8235-46d4-95e7-69caf9b93e91"
-					(reference "D5")
+					(reference "D7")
 					(unit 1)
 				)
@@
 		(dnp no)
 		(fields_autoplaced yes)
-		(property "Reference" "D6"
+		(property "Reference" "D5"
 			(at 250.19 82.5499 90)
 			(show_name no)
@@
 			(project "Electronic Trombone"
 				(path "/931827f3-33b7-460f-8885-7db258da2648/6d65ef8f-8235-46d4-95e7-69caf9b93e91"
-					(reference "D6")
+					(reference "D5")
 					(unit 1)
 				)
@@
 		(dnp no)
 		(fields_autoplaced yes)
-		(property "Reference" "D8"
+		(property "Reference" "D9"
 			(at 71.12 92.7099 90)
 			(show_name no)
@@
 			(project "Electronic Trombone"
 				(path "/931827f3-33b7-460f-8885-7db258da2648/6d65ef8f-8235-46d4-95e7-69caf9b93e91"
-					(reference "D8")
+					(reference "D9")
 					(unit 1)
 				)
@@
 		(at 189.23 53.34 0)
 		(mirror x)
-		(unit 2)
+		(unit 4)
 		(body_style 1)
 		(exclude_from_sim no)
@@
 				(path "/931827f3-33b7-460f-8885-7db258da2648/6d65ef8f-8235-46d4-95e7-69caf9b93e91"
 					(reference "U7")
-					(unit 2)
+					(unit 4)
 				)
 			)
@@
 		(dnp no)
 		(fields_autoplaced yes)
-		(property "Reference" "D9"
+		(property "Reference" "D6"
 			(at 250.19 95.2499 90)
 			(show_name no)
@@
 			(project "Electronic Trombone"
 				(path "/931827f3-33b7-460f-8885-7db258da2648/6d65ef8f-8235-46d4-95e7-69caf9b93e91"
-					(reference "D9")
+					(reference "D6")
 					(unit 1)
 				)

Commit message: routed the filter, updated 0201 footprints to 0402
JLCPCB's economy PCBA has a footprint bottom limit of 0402 imperial
Parts:
- R37, R38, R40, R42, R44, R45, R47: footprint Resistor_SMD:R_0201_0603Metric -> Resistor_SMD:R_0402_1005Metric
Connections:
- net Unprocessed Out: now also U8.12 (+); no longer U8.3 (+)
- new net: R49.1, U8.13 (-), U8.14
Changed lines of the file:
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@@
 			)
 		)
-		(property "Footprint" "Resistor_SMD:R_0201_0603Metric"
+		(property "Footprint" "Resistor_SMD:R_0402_1005Metric"
 			(at 189.484 42.164 90)
 			(hide yes)
@@
 			)
 		)
-		(property "Footprint" "Resistor_SMD:R_0201_0603Metric"
+		(property "Footprint" "Resistor_SMD:R_0402_1005Metric"
 			(at 170.434 64.516 90)
 			(hide yes)
@@
 			)
 		)
-		(property "Footprint" "Resistor_SMD:R_0201_0603Metric"
+		(property "Footprint" "Resistor_SMD:R_0402_1005Metric"
 			(at 165.354 91.694 90)
 			(hide yes)
@@
 		(lib_id "Amplifier_Operational:TL074")
 		(at 45.72 152.4 0)
-		(unit 1)
+		(unit 4)
 		(body_style 1)
 		(exclude_from_sim no)
@@
 				(path "/931827f3-33b7-460f-8885-7db258da2648/6d65ef8f-8235-46d4-95e7-69caf9b93e91"
 					(reference "U8")
-					(unit 1)
+					(unit 4)
 				)
 			)
@@
 			)
 		)
-		(property "Footprint" "Resistor_SMD:R_0201_0603Metric"
+		(property "Footprint" "Resistor_SMD:R_0402_1005Metric"
 			(at 189.484 87.884 90)
 			(hide yes)
@@
 			)
 		)
-		(property "Footprint" "Resistor_SMD:R_0201_0603Metric"
+		(property "Footprint" "Resistor_SMD:R_0402_1005Metric"
 			(at 165.354 101.854 90)
 			(hide yes)
@@
 			)
 		)
-		(property "Footprint" "Resistor_SMD:R_0201_0603Metric"
+		(property "Footprint" "Resistor_SMD:R_0402_1005Metric"
 			(at 170.434 74.676 90)
 			(hide yes)
@@
 			)
 		)
-		(property "Footprint" "Resistor_SMD:R_0201_0603Metric"
+		(property "Footprint" "Resistor_SMD:R_0402_1005Metric"
 			(at 176.784 49.784 90)
 			(hide yes)

Commit message: all SMD are 0603 (imperial) now, started rerouting all traces
Parts:
- R37, R38, R39, R40, R42, R44, R45, R46, R47: footprint Resistor_SMD:R_0402_1005Metric -> Resistor_SMD:R_0603_1608Metric
Connections:
- net GND: now also U7.3 (+); no longer U7.10 (+)
- net Processed Control: now also U7.8, U7.9 (-); no longer U7.6 (-), U7.7
- net at D7.2 (A), R41.1, R43.2: now also U7.10 (+); no longer U7.5 (+)
- net at R44.1, R45.2, R47.2: now also U7.2 (-); no longer U7.9 (-)
- net at R46.2: now also U7.1; no longer U7.8
