File: KiCad/Custom Potentiometer Controls.kicad_sch (KiCad schematic)
At the start: 20 parts, among them J2 691137710003, J5 691137710002, U1 CD74HC4051E, U11 TL074

Commit message: placed and routed custom pot control
Parts:
- added C32, C33: 0.1u, Capacitor_SMD:C_0201_0603Metric, symbol Device:C_Small
Connections:
- net +5V: now also U11.13 (-), U11.14, C32.2; no longer U11.1, U11.2 (-)
- net +Pot: now also R2.1
- net -5V: now also U11.1, U11.2 (-), C33.1; no longer U11.13 (-), U11.14
- net GND: now also C32.1, C33.2
- net Mux Out: no longer R2.1
- net Trigger 1: now also J2.3; no longer J2.1
- net Trigger 3: now also J2.1; no longer J2.3
- net at R71.1, R73.2: now also U11.3 (+); no longer U11.12 (+)
- net at R72.1, R74.2: now also U11.12 (+); no longer U11.3 (+)
Other:
- moved on the sheet: R1, R2, R3, R4, RV14, U11B, U11C

Commit message: routed oscillator
Parts:
- added J6: 691137710002, Header 691137710002:691137710002, symbol Header 691137710002:691137710002
Connections:
- net +5V: now also J6.1
- net GND: now also J6.2
Other:
- note added: "To allow the button controls PCB to get the +5V source"

Commit message: routed the filter, updated 0201 footprints to 0402
JLCPCB's economy PCBA has a footprint bottom limit of 0402 imperial
Parts:
- C32, C33: footprint Capacitor_SMD:C_0201_0603Metric -> Capacitor_SMD:C_0402_1005Metric
- R1, R2, R3, R4, R71, R72, R73, R74: footprint Resistor_SMD:R_0201_0603Metric -> Resistor_SMD:R_0402_1005Metric
Changed lines of the file:
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@@
 			)
 		)
-		(property "Footprint" "Resistor_SMD:R_0201_0603Metric"
+		(property "Footprint" "Resistor_SMD:R_0402_1005Metric"
 			(at 62.484 26.416 90)
 			(hide yes)
@@
 			)
 		)
-		(property "Footprint" "Resistor_SMD:R_0201_0603Metric"
+		(property "Footprint" "Resistor_SMD:R_0402_1005Metric"
 			(at 109.474 185.166 90)
 			(hide yes)
@@
 			)
 		)
-		(property "Footprint" "Resistor_SMD:R_0201_0603Metric"
+		(property "Footprint" "Resistor_SMD:R_0402_1005Metric"
 			(at 119.634 161.544 90)
 			(hide yes)
@@
 			)
 		)
-		(property "Footprint" "Resistor_SMD:R_0201_0603Metric"
+		(property "Footprint" "Resistor_SMD:R_0402_1005Metric"
 			(at 105.664 161.544 90)
 			(hide yes)
@@
 			)
 		)
-		(property "Footprint" "Resistor_SMD:R_0201_0603Metric"
+		(property "Footprint" "Resistor_SMD:R_0402_1005Metric"
 			(at 62.484 34.036 90)
 			(hide yes)
@@
 			)
 		)
-		(property "Footprint" "Resistor_SMD:R_0201_0603Metric"
+		(property "Footprint" "Resistor_SMD:R_0402_1005Metric"
 			(at 20.574 35.306 90)
 			(hide yes)
@@
 			)
 		)
-		(property "Footprint" "Resistor_SMD:R_0201_0603Metric"
+		(property "Footprint" "Resistor_SMD:R_0402_1005Metric"
 			(at 20.574 27.686 90)
 			(hide yes)
@@
 			)
 		)
-		(property "Footprint" "Capacitor_SMD:C_0201_0603Metric"
+		(property "Footprint" "Capacitor_SMD:C_0402_1005Metric"
 			(at 83.82 113.03 0)
 			(hide yes)
@@
 			)
 		)
-		(property "Footprint" "Resistor_SMD:R_0201_0603Metric"
+		(property "Footprint" "Resistor_SMD:R_0402_1005Metric"
 			(at 105.664 171.704 90)
 			(hide yes)
@@
 			)
 		)
-		(property "Footprint" "Capacitor_SMD:C_0201_0603Metric"
+		(property "Footprint" "Capacitor_SMD:C_0402_1005Metric"
 			(at 149.86 77.47 0)
 			(hide yes)

Commit message: all SMD are 0603 (imperial) now, started rerouting all traces
Parts:
- C32, C33: footprint Capacitor_SMD:C_0402_1005Metric -> Capacitor_SMD:C_0603_1608Metric
- R1, R2, R3, R4, R71, R72, R73, R74: footprint Resistor_SMD:R_0402_1005Metric -> Resistor_SMD:R_0603_1608Metric
