File: KiCad/Power.kicad_sch (KiCad schematic)
At the start: 33 parts, among them SW4 SW_DPST, U10 TL074, U11 TL074, U2 TL074, U3 TL074, U4 40106, U5 TL074, U6 TL074, U7 TL074, U8 TL074, U9 TL074

Commit message: routed rest of the envelope generator
Connections:
- net GND: now also U3.10 (+); no longer U3.5 (+)
- net Thaw 3: now also U3.8, U3.9 (-); no longer U3.6 (-), U3.7
Changed lines of the file:
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@@
 		(lib_id "Amplifier_Operational:TL074")
 		(at 105.41 105.41 0)
-		(unit 2)
+		(unit 3)
 		(body_style 1)
 		(exclude_from_sim no)
@@
 				(path "/3ca3a63e-46c1-4b14-be30-fce478aad491"
 					(reference "U3")
-					(unit 2)
+					(unit 3)
 				)
 			)

Commit message: all SMD are 0603 (imperial) now, started rerouting all traces
Parts:
- C12, C13, C14, C15, C16, C17, C18, C19, C20, C21, C22, C23, C24, C25, C26, C27, C28, C29, C30, C31: footprint Capacitor_SMD:C_0402_1005Metric -> Capacitor_SMD:C_0603_1608Metric
Connections:
- net GND: now also U5.3 (+), U5.5 (+); no longer U5.10 (+), U5.12 (+)
- net Thaw 5C: now also U5.1, U5.2 (-); no longer U5.8, U5.9 (-)
- net Thaw 5D: now also U5.6 (-), U5.7; no longer U5.13 (-), U5.14

Commit message: first JLCPCB order
Connections:
- net GND: now also U2.5 (+); no longer U2.3 (+)
- net Thaw 2: now also U2.6 (-), U2.7; no longer U2.1, U2.2 (-)
Changed lines of the file:
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@@
 		(lib_id "Amplifier_Operational:TL074")
 		(at 77.47 105.41 0)
-		(unit 1)
+		(unit 2)
 		(body_style 1)
 		(exclude_from_sim no)
@@
 				(path "/3ca3a63e-46c1-4b14-be30-fce478aad491"
 					(reference "U2")
-					(unit 1)
+					(unit 2)
 				)
 			)
