File: KiCad/Oscillator/Electronic Trombone Oscillator.kicad_sch (KiCad schematic)
At the start: 12 parts, among them J1 691137710002, U2 TL074, U3 TL074

Commit message: started separating into different boards, partially fixed envelope generator
Parts:
- removed R5, R6: R_US, Resistor_THT:R_Axial_DIN0207_L6.3mm_D2.5mm_P7.62mm_Horizontal, symbol Device:R_US
- removed RV8: 100k, Potentiometer 100k PTV09A-2020F-B104:Potentiometer 100k PTV09A-2020F-B104, symbol Device:R_Potentiometer_US
- removed unit 4 of U2
- removed unit 1 of U2
Other:
- removed sheet Amplifier
- removed sheet Filter
- note added: "Req. 0V to -2V"
- note added: "Simulated up to 6.3V"
- note added: "Simulated up to 8.3V"
- note removed: "10mV pp."
