File: KiCad/Oscillator/Oscillator.kicad_sch (KiCad schematic)
At the start: 57 parts, among them J1 Screw_Terminal_01x02, J2 Screw_Terminal_01x03, Q1 NPN, Q2 PNP, Q3 NPN, Q4 PNP, U1 40106, U2 TL074, U3 TL074

Commit message: added power indicator LEDs
Parts:
- gave numbers to parts that had none: 21
Changed lines of the file:
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@@
 		(in_pos_files yes)
 		(dnp no)
-		(property "Reference" "TP?"
+		(property "Reference" "TP5"
 			(at 31.75 49.53 0)
 			(hide yes)
@@
 			(project "Oscillator"
 				(path "/931827f3-33b7-460f-8885-7db258da2648"
-					(reference "TP?")
+					(reference "TP5")
 					(unit 1)
 				)
@@
 		(in_pos_files yes)
 		(dnp no)
-		(property "Reference" "TP?"
+		(property "Reference" "TP4"
 			(at 233.68 48.26 0)
 			(hide yes)
@@
 			(project "Oscillator"
 				(path "/931827f3-33b7-460f-8885-7db258da2648"
-					(reference "TP?")
+					(reference "TP4")
 					(unit 1)
 				)
@@
 		(dnp no)
 		(fields_autoplaced yes)
-		(property "Reference" "#PWR08"
+		(property "Reference" "#PWR07"
 			(at 109.22 69.85 0)
 			(hide yes)
@@
 			(project "Oscillator"
 				(path "/931827f3-33b7-460f-8885-7db258da2648"
-					(reference "#PWR08")
+					(reference "#PWR07")
 					(unit 1)
 				)
@@
 		(in_pos_files yes)
 		(dnp no)
-		(property "Reference" "TP?"
+		(property "Reference" "TP21"
 			(at 76.2 147.32 0)
 			(hide yes)
@@
 			(project "Oscillator"
 				(path "/931827f3-33b7-460f-8885-7db258da2648"
-					(reference "TP?")
+					(reference "TP21")
 					(unit 1)
 				)
@@
 		(in_pos_files yes)
 		(dnp no)
-		(property "Reference" "TP?"
+		(property "Reference" "TP19"
 			(at 31.75 139.7 0)
 			(hide yes)
@@
 			(project "Oscillator"
 				(path "/931827f3-33b7-460f-8885-7db258da2648"
-					(reference "TP?")
+					(reference "TP19")
 					(unit 1)
 				)
@@
 		(in_pos_files yes)
 		(dnp no)
-		(property "Reference" "TP?"
+		(property "Reference" "TP12"
 			(at 76.2 69.8216 0)
 			(hide yes)
@@
 			(project "Oscillator"
 				(path "/931827f3-33b7-460f-8885-7db258da2648"
-					(reference "TP?")
+					(reference "TP12")
 					(unit 1)
 				)
@@
 		(dnp no)
 		(fields_autoplaced yes)
-		(property "Reference" "#PWR03"
+		(property "Reference" "#PWR02"
 			(at 109.22 41.91 0)
 			(hide yes)
@@
 			(project "Oscillator"
 				(path "/931827f3-33b7-460f-8885-7db258da2648"
-					(reference "#PWR03")
+					(reference "#PWR02")
 					(unit 1)
 				)
@@
 		(in_pos_files yes)
 		(dnp no)
-		(property "Reference" "TP?"
+		(property "Reference" "TP9"
 			(at 31.75 62.23 0)
 			(hide yes)
@@
 			(project "Oscillator"
 				(path "/931827f3-33b7-460f-8885-7db258da2648"
-					(reference "TP?")
+					(reference "TP9")
 					(unit 1)
 				)
@@
 		(in_pos_files yes)
 		(dnp no)
-		(property "Reference" "TP?"
+		(property "Reference" "TP3"
 			(at 31.75 36.83 0)
 			(hide yes)
@@
 			(project "Oscillator"
 				(path "/931827f3-33b7-460f-8885-7db258da2648"
-					(reference "TP?")
+					(reference "TP3")
 					(unit 1)
 				)
@@
 		(dnp no)
 		(fields_autoplaced yes)
-		(property "Reference" "#PWR016"
+		(property "Reference" "#PWR015"
 			(at 109.22 119.38 0)
 			(hide yes)
@@
 			(project "Oscillator"
 				(path "/931827f3-33b7-460f-8885-7db258da2648"
-					(reference "#PWR016")
+					(reference "#PWR015")
 					(unit 1)
 				)
@@
 		(in_pos_files yes)
 		(dnp no)
-		(property "Reference" "TP?"
+		(property "Reference" "TP8"
 			(at 76.2 57.15 0)
 			(hide yes)
@@
 			(project "Oscillator"
 				(path "/931827f3-33b7-460f-8885-7db258da2648"
-					(reference "TP?")
+					(reference "TP8")
 					(unit 1)
 				)
@@
 		(dnp no)
 		(fields_autoplaced yes)
-		(property "Reference" "#PWR02"
+		(property "Reference" "#PWR03"
 			(at 30.48 35.56 0)
 			(hide yes)
@@
 			(project "Oscillator"
 				(path "/931827f3-33b7-460f-8885-7db258da2648"
-					(reference "#PWR02")
+					(reference "#PWR03")
 					(unit 1)
 				)
@@
 		(in_pos_files yes)
 		(dnp no)
-		(property "Reference" "TP?"
+		(property "Reference" "TP6"
 			(at 233.68 50.8 0)
 			(hide yes)
@@
 			(project "Oscillator"
 				(path "/931827f3-33b7-460f-8885-7db258da2648"
-					(reference "TP?")
+					(reference "TP6")
 					(unit 1)
 				)
@@
 		(in_pos_files yes)
 		(dnp no)
-		(property "Reference" "TP?"
+		(property "Reference" "TP10"
 			(at 179.07 62.23 0)
 			(hide yes)
@@
 			(project "Oscillator"
 				(path "/931827f3-33b7-460f-8885-7db258da2648"
-					(reference "TP?")
+					(reference "TP10")
 					(unit 1)
 				)
@@
 		(in_pos_files yes)
 		(dnp no)
-		(property "Reference" "TP?"
+		(property "Reference" "TP7"
 			(at 38.1 57.15 0)
 			(hide yes)
@@
 			(project "Oscillator"
 				(path "/931827f3-33b7-460f-8885-7db258da2648"
-					(reference "TP?")
+					(reference "TP7")
 					(unit 1)
 				)
@@
 		(in_pos_files yes)
 		(dnp no)
-		(property "Reference" "TP?"
+		(property "Reference" "TP17"
 			(at 38.1 134.62 0)
 			(hide yes)
@@
 			(project "Oscillator"
 				(path "/931827f3-33b7-460f-8885-7db258da2648"
-					(reference "TP?")
+					(reference "TP17")
 					(unit 1)
 				)
@@
 		(in_pos_files yes)
 		(dnp no)
-		(property "Reference" "TP?"
+		(property "Reference" "TP13"
 			(at 31.75 101.6 0)
 			(hide yes)
@@
 			(project "Oscillator"
 				(path "/931827f3-33b7-460f-8885-7db258da2648"
-					(reference "TP?")
+					(reference "TP13")
 					(unit 1)
 				)
@@
 		(in_pos_files yes)
 		(dnp no)
-		(property "Reference" "TP?"
+		(property "Reference" "TP18"
 			(at 76.2 134.62 0)
 			(hide yes)
@@
 			(project "Oscillator"
 				(path "/931827f3-33b7-460f-8885-7db258da2648"
-					(reference "TP?")
+					(reference "TP18")
 					(unit 1)
 				)
@@
 		(in_pos_files yes)
 		(dnp no)
-		(property "Reference" "TP?"
+		(property "Reference" "TP11"
 			(at 233.68 64.77 0)
 			(hide yes)
@@
 			(project "Oscillator"
 				(path "/931827f3-33b7-460f-8885-7db258da2648"
-					(reference "TP?")
+					(reference "TP11")
 					(unit 1)
 				)
@@
 		(dnp no)
 		(fields_autoplaced yes)
-		(property "Reference" "#PWR020"
+		(property "Reference" "#PWR021"
 			(at 30.48 138.43 0)
 			(hide yes)
@@
 			(project "Oscillator"
 				(path "/931827f3-33b7-460f-8885-7db258da2648"
-					(reference "#PWR020")
+					(reference "#PWR021")
 					(unit 1)
 				)
@@
 		(dnp no)
 		(fields_autoplaced yes)
-		(property "Reference" "#PWR015"
+		(property "Reference" "#PWR016"
 			(at 30.48 113.03 0)
 			(hide yes)
@@
 			(project "Oscillator"
 				(path "/931827f3-33b7-460f-8885-7db258da2648"
-					(reference "#PWR015")
+					(reference "#PWR016")
 					(unit 1)
 				)
@@
 		(in_pos_files yes)
 		(dnp no)
-		(property "Reference" "TP?"
+		(property "Reference" "TP2"
 			(at 38.1 31.75 0)
 			(hide yes)
@@
 			(project "Oscillator"
 				(path "/931827f3-33b7-460f-8885-7db258da2648"
-					(reference "TP?")
+					(reference "TP2")
 					(unit 1)
 				)
@@
 		(dnp no)
 		(fields_autoplaced yes)
-		(property "Reference" "#PWR021"
+		(property "Reference" "#PWR020"
 			(at 109.22 147.32 0)
 			(hide yes)
@@
 			(project "Oscillator"
 				(path "/931827f3-33b7-460f-8885-7db258da2648"
-					(reference "#PWR021")
+					(reference "#PWR020")
 					(unit 1)
 				)
@@
 		(in_pos_files yes)
 		(dnp no)
-		(property "Reference" "TP?"
+		(property "Reference" "TP15"
 			(at 31.75 114.3 0)
 			(hide yes)
@@
 			(project "Oscillator"
 				(path "/931827f3-33b7-460f-8885-7db258da2648"
-					(reference "TP?")
+					(reference "TP15")
 					(unit 1)
 				)
@@
 		(in_pos_files yes)
 		(dnp no)
-		(property "Reference" "TP?"
+		(property "Reference" "TP16"
 			(at 31.75 127 0)
 			(hide yes)
@@
 			(project "Oscillator"
 				(path "/931827f3-33b7-460f-8885-7db258da2648"
-					(reference "TP?")
+					(reference "TP16")
 					(unit 1)
 				)
@@
 		(in_pos_files yes)
 		(dnp no)
-		(property "Reference" "TP?"
+		(property "Reference" "TP14"
 			(at 38.1 109.22 0)
 			(hide yes)
@@
 			(project "Oscillator"
 				(path "/931827f3-33b7-460f-8885-7db258da2648"
-					(reference "TP?")
+					(reference "TP14")
 					(unit 1)
 				)
@@
 		(dnp no)
 		(fields_autoplaced yes)
-		(property "Reference" "#PWR09"
+		(property "Reference" "#PWR08"
 			(at 233.68 67.31 0)
 			(hide yes)
@@
 			(project "Oscillator"
 				(path "/931827f3-33b7-460f-8885-7db258da2648"
-					(reference "#PWR09")
+					(reference "#PWR08")
 					(unit 1)
 				)
@@
 		(in_pos_files yes)
 		(dnp no)
-		(property "Reference" "TP?"
+		(property "Reference" "TP1"
 			(at 31.75 24.13 0)
 			(hide yes)
@@
 			(project "Oscillator"
 				(path "/931827f3-33b7-460f-8885-7db258da2648"
-					(reference "TP?")
+					(reference "TP1")
 					(unit 1)
 				)
@@
 		(in_pos_files yes)
 		(dnp no)
-		(property "Reference" "TP?"
+		(property "Reference" "TP20"
 			(at 179.07 139.7 0)
 			(hide yes)
@@
 			(project "Oscillator"
 				(path "/931827f3-33b7-460f-8885-7db258da2648"
-					(reference "TP?")
+					(reference "TP20")
 					(unit 1)
 				)
@@
 		(dnp no)
 		(fields_autoplaced yes)
-		(property "Reference" "#PWR07"
+		(property "Reference" "#PWR09"
 			(at 30.48 60.96 0)
 			(hide yes)
@@
 			(project "Oscillator"
 				(path "/931827f3-33b7-460f-8885-7db258da2648"
-					(reference "#PWR07")
+					(reference "#PWR09")
 					(unit 1)
 				)

Commit message: updated footprints in oscillator
Parts:
- J1: footprint (none) -> Header 691137710002:691137710002
- J2: footprint (none) -> Header 691137710003:691137710003
- R1, R2, R3, R4, R5, R6, R7, R8: footprint Resistor_SMD:R_0603_1608Metric -> Resistor_SMD:R_0805_2012Metric
- RV1, RV3, RV5, RV6, RV8: footprint (none) -> Potentiometer_THT:Potentiometer_Bourns_3339P_Vertical_HandSoldering
- RV2, RV4, RV7: footprint Potentiometer 100k PTV09A-2020F-B104:Potentiometer 100k PTV09A-2020F-B104 -> Potentiometer_THT:Potentiometer_Bourns_PTV09A-2_Single_Horizontal
- TP1, TP10, TP11, TP12, TP13, TP14, TP15, TP16, TP17, TP18, TP19, TP2, TP20, TP21, TP3, TP4, TP5, TP6, TP7, TP8, TP9: footprint (none) -> TestPoint:TestPoint_Keystone_5000-5004_Miniature
- U1: footprint Schmitt Inv. CD40106BE:N14 -> Package_DIP:DIP-14_W7.62mm
Changed lines of the file:
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@@
 			)
 		)
-		(property "Footprint" "Resistor_SMD:R_0603_1608Metric"
+		(property "Footprint" "Resistor_SMD:R_0805_2012Metric"
 			(at 110.236 42.164 90)
 			(hide yes)
@@
 			)
 		)
-		(property "Footprint" "Potentiometer 100k PTV09A-2020F-B104:Potentiometer 100k PTV09A-2020F-B104"
+		(property "Footprint" "Potentiometer_THT:Potentiometer_Bourns_PTV09A-2_Single_Horizontal"
 			(at 30.48 58.42 0)
 			(hide yes)
@@
 			)
 		)
-		(property "Footprint" "Schmitt Inv. CD40106BE:N14"
+		(property "Footprint" "Package_DIP:DIP-14_W7.62mm"
 			(at 152.4 44.45 0)
 			(hide yes)
@@
 			)
 		)
-		(property "Footprint" ""
+		(property "Footprint" "Header 691137710002:691137710002"
 			(at 238.76 49.53 0)
 			(hide yes)
@@
 			)
 		)
-		(property "Footprint" ""
+		(property "Footprint" "TestPoint:TestPoint_Keystone_5000-5004_Miniature"
 			(at 35.56 50.8 0)
 			(hide yes)
@@
 			)
 		)
-		(property "Footprint" ""
+		(property "Footprint" "TestPoint:TestPoint_Keystone_5000-5004_Miniature"
 			(at 237.49 49.53 0)
 			(hide yes)
@@
 			)
 		)
-		(property "Footprint" ""
+		(property "Footprint" "TestPoint:TestPoint_Keystone_5000-5004_Miniature"
 			(at 80.01 148.59 0)
 			(hide yes)
@@
 			)
 		)
-		(property "Footprint" "Resistor_SMD:R_0603_1608Metric"
+		(property "Footprint" "Resistor_SMD:R_0805_2012Metric"
 			(at 43.434 57.404 90)
 			(hide yes)
@@
 			)
 		)
-		(property "Footprint" "Resistor_SMD:R_0603_1608Metric"
+		(property "Footprint" "Resistor_SMD:R_0805_2012Metric"
 			(at 43.434 80.264 90)
 			(hide yes)
@@
 			)
 		)
-		(property "Footprint" ""
+		(property "Footprint" "TestPoint:TestPoint_Keystone_5000-5004_Miniature"
 			(at 35.56 140.97 0)
 			(hide yes)
@@
 			)
 		)
-		(property "Footprint" ""
+		(property "Footprint" "Header 691137710003:691137710003"
 			(at 238.76 66.04 0)
 			(hide yes)
@@
 			)
 		)
-		(property "Footprint" ""
+		(property "Footprint" "TestPoint:TestPoint_Keystone_5000-5004_Miniature"
 			(at 80.01 71.0916 0)
 			(hide yes)
@@
 			)
 		)
-		(property "Footprint" ""
+		(property "Footprint" "TestPoint:TestPoint_Keystone_5000-5004_Miniature"
 			(at 35.56 63.5 0)
 			(hide yes)
@@
 			)
 		)
-		(property "Footprint" ""
+		(property "Footprint" "TestPoint:TestPoint_Keystone_5000-5004_Miniature"
 			(at 35.56 38.1 0)
 			(hide yes)
@@
 			)
 		)
-		(property "Footprint" ""
+		(property "Footprint" "Potentiometer_THT:Potentiometer_Bourns_3339P_Vertical_HandSoldering"
 			(at 74.93 143.51 0)
 			(hide yes)
@@
 			)
 		)
-		(property "Footprint" ""
+		(property "Footprint" "TestPoint:TestPoint_Keystone_5000-5004_Miniature"
 			(at 80.01 58.42 0)
 			(hide yes)
@@
 			)
 		)
-		(property "Footprint" ""
+		(property "Footprint" "TestPoint:TestPoint_Keystone_5000-5004_Miniature"
 			(at 237.49 52.07 0)
 			(hide yes)
@@
 			)
 		)
-		(property "Footprint" ""
+		(property "Footprint" "TestPoint:TestPoint_Keystone_5000-5004_Miniature"
 			(at 182.88 63.5 0)
 			(hide yes)
@@
 			)
 		)
-		(property "Footprint" ""
+		(property "Footprint" "TestPoint:TestPoint_Keystone_5000-5004_Miniature"
 			(at 41.91 58.42 0)
 			(hide yes)
@@
 			)
 		)
-		(property "Footprint" "Schmitt Inv. CD40106BE:N14"
+		(property "Footprint" "Package_DIP:DIP-14_W7.62mm"
 			(at 152.4 121.92 0)
 			(hide yes)
@@
 			)
 		)
-		(property "Footprint" ""
+		(property "Footprint" "TestPoint:TestPoint_Keystone_5000-5004_Miniature"
 			(at 41.91 135.89 0)
 			(hide yes)
@@
 			)
 		)
-		(property "Footprint" ""
+		(property "Footprint" "TestPoint:TestPoint_Keystone_5000-5004_Miniature"
 			(at 35.56 102.87 0)
 			(hide yes)
@@
 			)
 		)
-		(property "Footprint" ""
+		(property "Footprint" "TestPoint:TestPoint_Keystone_5000-5004_Miniature"
 			(at 80.01 135.89 0)
 			(hide yes)
@@
 			)
 		)
-		(property "Footprint" ""
+		(property "Footprint" "Potentiometer_THT:Potentiometer_Bourns_3339P_Vertical_HandSoldering"
 			(at 30.48 33.02 0)
 			(hide yes)
@@
 			)
 		)
-		(property "Footprint" "Resistor_SMD:R_0603_1608Metric"
+		(property "Footprint" "Resistor_SMD:R_0805_2012Metric"
 			(at 110.236 119.634 90)
 			(hide yes)
@@
 			)
 		)
-		(property "Footprint" ""
+		(property "Footprint" "TestPoint:TestPoint_Keystone_5000-5004_Miniature"
 			(at 237.49 66.04 0)
 			(hide yes)
@@
 			)
 		)
-		(property "Footprint" "Resistor_SMD:R_0603_1608Metric"
+		(property "Footprint" "Resistor_SMD:R_0805_2012Metric"
 			(at 43.434 32.004 90)
 			(hide yes)
@@
 			)
 		)
-		(property "Footprint" "Potentiometer 100k PTV09A-2020F-B104:Potentiometer 100k PTV09A-2020F-B104"
+		(property "Footprint" "Potentiometer_THT:Potentiometer_Bourns_PTV09A-2_Single_Horizontal"
 			(at 30.48 135.89 0)
 			(hide yes)
@@
 			)
 		)
-		(property "Footprint" ""
+		(property "Footprint" "TestPoint:TestPoint_Keystone_5000-5004_Miniature"
 			(at 41.91 33.02 0)
 			(hide yes)
@@
 			)
 		)
-		(property "Footprint" "Resistor_SMD:R_0603_1608Metric"
+		(property "Footprint" "Resistor_SMD:R_0805_2012Metric"
 			(at 43.434 134.874 90)
 			(hide yes)
@@
 			)
 		)
-		(property "Footprint" ""
+		(property "Footprint" "Potentiometer_THT:Potentiometer_Bourns_3339P_Vertical_HandSoldering"
 			(at 213.36 101.6 0)
 			(hide yes)
@@
 			)
 		)
-		(property "Footprint" "Resistor_SMD:R_0603_1608Metric"
+		(property "Footprint" "Resistor_SMD:R_0805_2012Metric"
 			(at 43.434 109.474 90)
 			(hide yes)
@@
 			)
 		)
-		(property "Footprint" ""
+		(property "Footprint" "TestPoint:TestPoint_Keystone_5000-5004_Miniature"
 			(at 35.56 115.57 0)
 			(hide yes)
@@
 			)
 		)
-		(property "Footprint" "Potentiometer 100k PTV09A-2020F-B104:Potentiometer 100k PTV09A-2020F-B104"
+		(property "Footprint" "Potentiometer_THT:Potentiometer_Bourns_PTV09A-2_Single_Horizontal"
 			(at 177.8 99.06 0)
 			(hide yes)
@@
 			)
 		)
-		(property "Footprint" ""
+		(property "Footprint" "TestPoint:TestPoint_Keystone_5000-5004_Miniature"
 			(at 35.56 128.27 0)
 			(hide yes)
@@
 			)
 		)
-		(property "Footprint" ""
+		(property "Footprint" "TestPoint:TestPoint_Keystone_5000-5004_Miniature"
 			(at 41.91 110.49 0)
 			(hide yes)
@@
 			)
 		)
-		(property "Footprint" ""
+		(property "Footprint" "Potentiometer_THT:Potentiometer_Bourns_3339P_Vertical_HandSoldering"
 			(at 74.93 66.04 0)
 			(hide yes)
@@
 			)
 		)
-		(property "Footprint" ""
+		(property "Footprint" "Potentiometer_THT:Potentiometer_Bourns_3339P_Vertical_HandSoldering"
 			(at 30.48 110.49 0)
 			(hide yes)
@@
 			)
 		)
-		(property "Footprint" ""
+		(property "Footprint" "TestPoint:TestPoint_Keystone_5000-5004_Miniature"
 			(at 35.56 25.4 0)
 			(hide yes)
@@
 			)
 		)
-		(property "Footprint" ""
+		(property "Footprint" "TestPoint:TestPoint_Keystone_5000-5004_Miniature"
 			(at 182.88 140.97 0)
 			(hide yes)
@@
 			)
 		)
-		(property "Footprint" "Resistor_SMD:R_0603_1608Metric"
+		(property "Footprint" "Resistor_SMD:R_0805_2012Metric"
 			(at 43.434 157.734 90)
 			(hide yes)

Commit message: oscillator pcb layout done
Parts:
- removed TP1, TP12, TP13, TP14, TP15, TP16, TP17, TP18, TP19, TP2, TP21, TP3, TP5, TP7, TP8, TP9: TestPoint_Small, TestPoint:TestPoint_Keystone_5000-5004_Miniature, symbol Connector:TestPoint_Small
- renumbered U3 to U2
Connections:
- net -9V: now also RV1.1, RV2.1; no longer RV1.3, RV2.3
- net GND: now also RV1.3, RV2.3, RV8.3; no longer RV1.1, RV2.1, RV8.1
- net Mix In 1: now also U2.1, U2.2 (-); no longer U2.13 (-), U2.14
- net Mix In 2: now also U2.13 (-), U2.14; no longer U2.8, U2.9 (-)
- net Processed Control 2: now also RV8.1; no longer RV8.3
- net Sch Inv In 1: now also U1.5, U2.3 (+); no longer U1.1, U2.12 (+)
- net Sch Inv In 2: now also U2.12 (+); no longer U2.10 (+)
- net Sch Inv Out 1: now also U1.6; no longer U1.2
- net at RV4.2: now also U2.10 (+); no longer U2.5 (+)
- new net: C2.1, U2.8, U2.9 (-)
Other:
- moved on the sheet: RV8
