File: KiCad/Oscillator/Oscillator.kicad_pcb (KiCad board)
At the start: 2 copper layers, 78 x 73.5 mm, 52 parts, among them J1 Screw_Terminal_01x02, J2 Screw_Terminal_01x03, Q1 NPN, Q2 PNP, Q3 NPN, Q4 PNP, U1 40106, U2 TL074

Commit message: preparation to merge project back into one board
Parts:
- moved TP5 4.35 mm to (82.0, 96.1)
- renumbered TP10 to TP1, TP20 to TP2, TP4 to TP3, TP6 to TP4, TP11 to TP5
Changed lines of the file:
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@@
 			(drillshape 0)
 			(scaleselection 1)
-			(outputdirectory "../Production/Jul 8 2026/")
+			(outputdirectory "../../Build/Aug 20 2026/")
 		)
 	)
@@
 		(descr "Keystone THM Miniature Test Point 5000-5004, http://www.keyelco.com/product-pdf.cfm?p=1309")
 		(tags "Through Hole Mount Test Points")
-		(property "Reference" "TP10"
+		(property "Reference" "TP1"
 			(at 0 -2.5 0)
 			(layer "F.SilkS")
@@
 		(tags "LED")
 		(property "Reference" "D3"
-			(at -1 -4 0)
+			(at -3 -2.5 0)
 			(layer "F.SilkS")
 			(effects
@@
 		(descr "Keystone THM Miniature Test Point 5000-5004, http://www.keyelco.com/product-pdf.cfm?p=1309")
 		(tags "Through Hole Mount Test Points")
-		(property "Reference" "TP6"
+		(property "Reference" "TP4"
 			(at 0 -2.5 0)
 			(layer "F.SilkS")
@@
 		(tags "LED")
 		(property "Reference" "D4"
-			(at -0.96 -4 0)
+			(at -2.96 -2.5 0)
 			(layer "F.SilkS")
 			(effects
@@
 		(at 84 104)
 		(property "Reference" "J2"
-			(at 0 -5.135 0)
+			(at 9 3.5 0)
 			(layer "F.SilkS")
 			(effects
@@
 		(descr "Keystone THM Miniature Test Point 5000-5004, http://www.keyelco.com/product-pdf.cfm?p=1309")
 		(tags "Through Hole Mount Test Points")
-		(property "Reference" "TP20"
+		(property "Reference" "TP2"
 			(at 0 -2.5 0)
 			(layer "F.SilkS")
@@
 	(footprint "TestPoint:TestPoint_Keystone_5000-5004_Miniature"
 		(layer "F.Cu")
-		(at 77.65 96.1)
+		(at 82 96.1)
 		(descr "Keystone THM Miniature Test Point 5000-5004, http://www.keyelco.com/product-pdf.cfm?p=1309")
 		(tags "Through Hole Mount Test Points")
-		(property "Reference" "TP11"
+		(property "Reference" "TP5"
 			(at 0 -2.5 0)
 			(layer "F.SilkS")
@@
 		(descr "Keystone THM Miniature Test Point 5000-5004, http://www.keyelco.com/product-pdf.cfm?p=1309")
 		(tags "Through Hole Mount Test Points")
-		(property "Reference" "TP4"
+		(property "Reference" "TP3"
 			(at 0 -2.5 0)
 			(layer "F.SilkS")
@@
 		(at 68.5 104)
 		(property "Reference" "J1"
-			(at 0 -5.135 0)
+			(at -6.5 3.5 0)
 			(layer "F.SilkS")
 			(effects
@@
 		)
 	)
+	(gr_line
+		(start 83.2 97.5)
+		(end 83.2 97.8)
+		(stroke
+			(width 0.1)
+			(type default)
+		)
+		(layer "F.SilkS")
+	)
+	(gr_line
+		(start 83.5 97.5)
+		(end 83.2 97.5)
+		(stroke
+			(width 0.1)
+			(type default)
+		)
+		(layer "F.SilkS")
+	)
+	(gr_line
+		(start 83.7 98)
+		(end 83.2 97.5)
+		(stroke
+			(width 0.1)
+			(type default)
+		)
+		(layer "F.SilkS")
+	)
 	(gr_arc
 		(start 40 39.5)
@@
 		(layer "Edge.Cuts")
 	)
+	(gr_text "+9V"
+		(at 78.5 99.5 0)
+		(layer "F.SilkS")
+		(effects
+			(font
+				(size 1 1)
+				(thickness 0.2)
+				(bold yes)
+			)
+			(justify bottom)
+		)
+	)
+	(gr_text "GND"
+		(at 84 99.5 0)
+		(layer "F.SilkS")
+		(effects
+			(font
+				(size 1 1)
+				(thickness 0.2)
+				(bold yes)
+			)
+			(justify bottom)
+		)
+	)
+	(gr_text "-9V"
+		(at 89 99.5 0)
+		(layer "F.SilkS")
+		(effects
+			(font
+				(size 1 1)
+				(thickness 0.2)
+				(bold yes)
+			)
+			(justify bottom)
+		)
+	)
 	(gr_text "Fine\nTune\n1"
 		(at 65 40.5 0)
@@
 	)
 	(gr_text "Control"
-		(at 67.6 93.5 0)
+		(at 65 100 0)
 		(layer "F.SilkS")
 		(effects
@@
 	)
 	(gr_text "Out"
-		(at 72.6 99.8 0)
-		(layer "F.SilkS")
-		(effects
-			(font
-				(size 1.5 1.5)
-				(thickness 0.3)
-				(bold yes)
-			)
-			(justify bottom)
-		)
-	)
-	(gr_text "GND"
-		(at 77.6 93.6 0)
+		(at 72.6 100 0)
 		(layer "F.SilkS")
 		(effects
