File: KiCad/Power/Power.kicad_pcb (KiCad board)
At the start: 2 copper layers, 97 x 98 mm, 49 parts, among them J1 Screw_Terminal_01x04, J2 Screw_Terminal_01x03, J3 Screw_Terminal_01x03, J4 Screw_Terminal_01x02, SW1 SW_DPST, U1 CD74HC4051E, U2 TL074, U3 L7805, U4 L7905

Commit message: added mounting holes to schematics, adjusted board sizes
Other:
- board text added: "Power"
