File: KiCad/Power/Power.kicad_pcb (KiCad board)
At the start: 2 copper layers, 100 x 90 mm, 50 parts, among them J1 Screw_Terminal_01x03, J2 Screw_Terminal_01x03, J3 Screw_Terminal_01x03, J4 Screw_Terminal_01x03, J5 Screw_Terminal_01x02, J6 Screw_Terminal_01x03, J7 Conn_01x03, J8 Screw_Terminal_01x02, SW1 SW_DPST, U1 CD74HC4051E, U2 TL074, U3 L7805, U4 L7905

Commit message: changed value of protective resistor in power board
Parts:
- R9: value 2.2k -> 1k
Changed lines of the file:
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@@
 			)
 		)
-		(property "Value" "2.2k"
+		(property "Value" "1k"
 			(at 0 1.65 0)
 			(layer "F.Fab")
@@
 	)
 	(segment
+		(start 108.4125 92.1025)
+		(end 107.12 90.81)
+		(width 0.25)
+		(layer "F.Cu")
+		(net "Net-(R4-Pad2)")
+	)
+	(segment
+		(start 104.5751 98.7)
+		(end 107.5 95.7751)
+		(width 0.25)
+		(layer "F.Cu")
+		(net "Net-(R4-Pad2)")
+	)
+	(segment
+		(start 108.4125 93.005)
+		(end 108.4125 92.1025)
+		(width 0.25)
+		(layer "F.Cu")
+		(net "Net-(R4-Pad2)")
+	)
+	(segment
+		(start 100.7125 98.7)
+		(end 104.5751 98.7)
+		(width 0.25)
+		(layer "F.Cu")
+		(net "Net-(R4-Pad2)")
+	)
+	(segment
+		(start 107.5 93.9175)
+		(end 108.4125 93.005)
+		(width 0.25)
+		(layer "F.Cu")
+		(net "Net-(R4-Pad2)")
+	)
+	(segment
+		(start 107.5 95.7751)
+		(end 107.5 93.9175)
+		(width 0.25)
+		(layer "F.Cu")
+		(net "Net-(R4-Pad2)")
+	)
+	(segment
+		(start 98.6875 99.1)
+		(end 98.7875 99.1)
+		(width 0.25)
+		(layer "F.Cu")
+		(net "/Pot -")
+	)
+	(segment
+		(start 98 99.5875)
+		(end 98.8875 98.7)
+		(width 0.25)
+		(layer "F.Cu")
+		(net "/Pot -")
+	)
+	(segment
+		(start 98 108.25)
+		(end 98 99.5875)
+		(width 0.25)
+		(layer "F.Cu")
+		(net "/Pot -")
+	)
+	(segment
 		(start 102 80.005)
 		(end 98.54 76.545)
@@
 	)
 	(segment
-		(start 98.6875 99.1)
-		(end 98.7875 99.1)
-		(width 0.25)
-		(layer "F.Cu")
-		(net "/Pot -")
-	)
-	(segment
-		(start 98 99.5875)
-		(end 98.8875 98.7)
-		(width 0.25)
-		(layer "F.Cu")
-		(net "/Pot -")
-	)
-	(segment
-		(start 98 108.25)
-		(end 98 99.5875)
-		(width 0.25)
-		(layer "F.Cu")
-		(net "/Pot -")
-	)
-	(segment
 		(start 109.25 85.32)
 		(end 107.12 83.19)
@@
 		(net "/Pot+ 4th Partial")
 	)
-	(segment
-		(start 108.4125 92.1025)
-		(end 107.12 90.81)
-		(width 0.25)
-		(layer "F.Cu")
-		(net "Net-(R4-Pad2)")
-	)
-	(segment
-		(start 104.5751 98.7)
-		(end 107.5 95.7751)
-		(width 0.25)
-		(layer "F.Cu")
-		(net "Net-(R4-Pad2)")
-	)
-	(segment
-		(start 108.4125 93.005)
-		(end 108.4125 92.1025)
-		(width 0.25)
-		(layer "F.Cu")
-		(net "Net-(R4-Pad2)")
-	)
-	(segment
-		(start 100.7125 98.7)
-		(end 104.5751 98.7)
-		(width 0.25)
-		(layer "F.Cu")
-		(net "Net-(R4-Pad2)")
-	)
-	(segment
-		(start 107.5 93.9175)
-		(end 108.4125 93.005)
-		(width 0.25)
-		(layer "F.Cu")
-		(net "Net-(R4-Pad2)")
-	)
-	(segment
-		(start 107.5 95.7751)
-		(end 107.5 93.9175)
-		(width 0.25)
-		(layer "F.Cu")
-		(net "Net-(R4-Pad2)")
-	)
 	(zone
