File: KiCad/Power/Power.kicad_pcb (KiCad board)
At the start: 2 copper layers, 100 x 90 mm, 50 parts, among them J1 Screw_Terminal_01x03, J2 Screw_Terminal_01x03, J3 Screw_Terminal_01x03, J4 Screw_Terminal_01x03, J5 Screw_Terminal_01x02, J6 Screw_Terminal_01x03, J7 Conn_01x03, J8 Screw_Terminal_01x02, SW1 SW_DPST, U1 CD74HC4051E, U2 TL074, U3 L7805, U4 L7905

Commit message: preparation to merge project back into one board
Parts:
- renumbered TP11 to TP3, TP12 to TP4, TP13 to TP5
Changed lines of the file:
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@@
 			(plot_on_all_layers_selection 0x00000000_00000000_00000000_00000000)
 			(disableapertmacros no)
-			(usegerberextensions no)
+			(usegerberextensions yes)
 			(usegerberattributes yes)
 			(usegerberadvancedattributes yes)
-			(creategerberjobfile yes)
+			(creategerberjobfile no)
 			(dashed_line_dash_ratio 12)
 			(dashed_line_gap_ratio 3)
@@
 			(outputformat 1)
 			(mirror no)
-			(drillshape 1)
+			(drillshape 0)
 			(scaleselection 1)
-			(outputdirectory "")
+			(outputdirectory "../../Build/Aug 20 2026/")
 		)
 	)
@@
 		(descr "Keystone THM Miniature Test Point 5000-5004, http://www.keyelco.com/product-pdf.cfm?p=1309")
 		(tags "Through Hole Mount Test Points")
-		(property "Reference" "TP12"
+		(property "Reference" "TP4"
 			(at 0 -2.5 0)
 			(layer "F.SilkS")
@@
 		(descr "Keystone THM Miniature Test Point 5000-5004, http://www.keyelco.com/product-pdf.cfm?p=1309")
 		(tags "Through Hole Mount Test Points")
-		(property "Reference" "TP13"
+		(property "Reference" "TP5"
 			(at 0 -2.5 0)
 			(layer "F.SilkS")
@@
 		(descr "Keystone THM Miniature Test Point 5000-5004, http://www.keyelco.com/product-pdf.cfm?p=1309")
 		(tags "Through Hole Mount Test Points")
-		(property "Reference" "TP11"
+		(property "Reference" "TP3"
 			(at 0 -2.5 0)
 			(layer "F.SilkS")

Commit message: merged project into one combined board (excluding the buttons)
Parts:
- renumbered C1 to C27, C2 to C28, C3 to C29, C4 to C30, D1 to D24, D2 to D25, D3 to D26, D4 to D27, H1 to H17, H2 to H18, H4 to H19, H3 to H20, J3 to J10, J2 to J11, J4 to J12, J5 to J13, J7 to J14, J6 to J15, J8 to J16, J1 to J9, R1 to R43, R2 to R44, R3 to R45, R4 to R46, R9 to R47, R5 to R48, R6 to R49, R7 to R50, R8 to R51, RV1 to RV25, RV2 to RV26, RV3 to RV27, RV4 to RV28, RV5 to RV29, RV6 to RV30, RV7 to RV31, RV8 to RV32, RV9 to RV33, TP3 to TP25, TP4 to TP26, TP5 to TP27, TP1 to TP28, TP2 to TP29, U3 to U10, U4 to U11, U1 to U8, U2 to U9
Other:
- board text removed: "+ LDO"
