File: KiCad/Power/Power.kicad_sch (KiCad schematic)
At the start: 50 parts, among them J1 Screw_Terminal_01x03, J2 Screw_Terminal_01x03, J3 Screw_Terminal_01x03, J4 Screw_Terminal_01x03, J5 Screw_Terminal_01x02, J6 Screw_Terminal_01x03, J7 Conn_01x03, J8 Screw_Terminal_01x02, SW1 SW_DPST, U1 CD74HC4051E, U2 TL074, U3 L7805, U4 L7905

Commit message: changed value of protective resistor in power board
Parts:
- R9: value 2.2k -> 1k
Changed lines of the file:
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@@
 			)
 		)
-		(property "Value" "2.2k"
+		(property "Value" "1k"
 			(at 105.41 170.18 90)
 			(show_name no)

Commit message: preparation to merge project back into one board
Parts:
- C1, C2, C3, C4, R1, R2, R3, R4, R5, R6, R7, R8, R9: KiLib_Generator (none) -> SMD_2terminal_chip_molded
- D1, D2, D3, D4: KiLib_Generator (none) -> LED/THT
- H1, H2, H3, H4: KiLib_Generator (none) -> mounting_hardware/mounting_hole
- J7: KiLib_Generator (none) -> connector/JST
- U1, U2: KiLib_Generator (none) -> package/DIP/legacy
- U3, U4: KiLib_Generator (none) -> package/TO_SOT/THT
