File: KiCad/Main/Main.kicad_sch (KiCad schematic)
At the start: 0 parts

Commit message: merged project into one combined board (excluding the buttons)
Parts:
- added C1, C3: 2.2n, Capacitor_THT:C_Rect_L18.0mm_W7.0mm_P15.00mm_FKS3_FKP3, symbol Device:C
- added C2: 1u, Capacitor_THT:C_Rect_L7.2mm_W4.5mm_P5.00mm, symbol Device:C
- added D1, D2: 1N4148, Diode_THT:D_DO-35_SOD27_P7.62mm_Horizontal, symbol Diode:1N4148
- added H1, H2, H3, H4: MountingHole, MountingHole:MountingHole_3.2mm_M3, symbol Mechanical:MountingHole
- added J1: Screw_Terminal_01x02, Header 691137710002:691137710002, symbol Connector:Screw_Terminal_01x02
- added J2: Screw_Terminal_01x03, Header 691137710003:691137710003, symbol Connector:Screw_Terminal_01x03
- added Q1, Q3: NPN, Package_TO_SOT_THT:TO-92, symbol Simulation_SPICE:NPN
- added Q2, Q4: PNP, Package_TO_SOT_THT:TO-92, symbol Simulation_SPICE:PNP
- added R1, R4, R5, R8: 100k, Resistor_SMD:R_0805_2012Metric, symbol Device:R_US
- added R2, R3, R6, R7: 1M, Resistor_SMD:R_0805_2012Metric, symbol Device:R_US
- added RV1, RV5, RV6: 100k, Potentiometer_THT:Potentiometer_Bourns_3339P_Vertical_HandSoldering, symbol Device:R_Potentiometer_Trim_US
- added RV2, RV4, RV7: 100k, Potentiometer_THT:Potentiometer_Bourns_PTV09A-2_Single_Horizontal, symbol Device:R_Potentiometer_US
- added RV3, RV8: 5k, Potentiometer_THT:Potentiometer_Bourns_3339P_Vertical_HandSoldering, symbol Device:R_Potentiometer_Trim_US
- added TH1, TH2, TH3, TH4, TH5, TH6: 10k, Resistor_THT:R_Radial_Power_L12.0mm_W8.0mm_P5.00mm, symbol Device:Thermistor_US
- added TP1, TP2, TP3, TP4, TP5: TestPoint_Small, TestPoint:TestPoint_Keystone_5000-5004_Miniature, symbol Connector:TestPoint_Small
- added U1: 40106, Package_DIP:DIP-14_W7.62mm, symbol 4xxx:40106
- added U2: TL074, Package_DIP:DIP-14_W7.62mm, symbol Amplifier_Operational:TL074
Connections:
- new net: Q1.2 (B), Q2.1 (C), R2.2
- new net: Q3.2 (B), Q4.1 (C), R6.2
- new net: R3.1, RV2.2
- new net: R3.2, TH2.1
- new net: R4.2, TH3.1
- new net: R1.2, TH1.1
- new net: R5.2, TH4.1
- new net: RV5.2, U2.5 (+)
- new net: R1.1, RV1.2
- new net: C2.1, U2.8, U2.9 (-)
- new net: C2.2, RV5.1
- new net: R8.2, TH6.1
- new net: R7.1, RV7.2
- new net: R7.2, TH5.1
- new net: R5.1, RV6.2
- new net: RV4.2, U2.10 (+)
- new net +9V: J2.1 (Pin_1), R2.1, R6.1
- new net -9V: J2.3 (Pin_3), RV1.1, RV2.1, RV6.3, RV7.3
- new net Control: J1.1 (Pin_1), R4.1, R8.1, TP3.1
- new net GND: C1.2, C3.2, J2.2 (Pin_2), Q1.3 (E), Q2.3 (E), Q3.3 (E), Q4.3 (E), RV1.3, RV2.3, RV3.1, RV5.3, RV6.1, RV7.1, RV8.3, TP5.1
- new net Mix In 1: RV4.3, TP1.1, U2.1, U2.2 (-)
- new net Mix In 2: RV4.1, TP2.1, U2.13 (-), U2.14
- new net Out: J1.2 (Pin_2), TP4.1, U2.6 (-), U2.7
- new net Processed Control 1: Q2.2 (B), RV3.2, RV3.3, TH1.2, TH2.2, TH3.2
- new net Processed Control 2: Q4.2 (B), RV8.1, RV8.2, TH4.2, TH5.2, TH6.2
- new net Sch Inv In 1: C1.1, D1.1 (K), Q1.1 (C), U1.5, U2.3 (+)
- new net Sch Inv In 2: C3.1, D2.1 (K), Q3.1 (C), U1.9, U2.12 (+)
- new net Sch Inv Out 1: D1.2 (A), U1.6
- new net Sch Inv Out 2: D2.2 (A), U1.8
Other:
- note added: "100mV pp., centered at 0V"
- note added: "Coarse Tuning"
- note added: "Fine Tuning"
