File: KiCad/Buttons/Buttons.kicad_pcb (KiCad board)
At the start: 2 copper layers, 19 x 69.5 mm, 13 parts, among them J1 691137710003, J2 691137710002

Commit message: preparation to merge project back into one board
Parts:
- renumbered TP7 to TP1, TP1 to TP2, TP4 to TP3, TP5 to TP4, TP6 to TP5
Changed lines of the file:
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@@
 			(plot_on_all_layers_selection 0x00000000_00000000_00000000_00000000)
 			(disableapertmacros no)
-			(usegerberextensions no)
+			(usegerberextensions yes)
 			(usegerberattributes yes)
 			(usegerberadvancedattributes yes)
-			(creategerberjobfile yes)
+			(creategerberjobfile no)
 			(dashed_line_dash_ratio 12)
 			(dashed_line_gap_ratio 3)
@@
 			(outputformat 1)
 			(mirror no)
-			(drillshape 1)
+			(drillshape 0)
 			(scaleselection 1)
-			(outputdirectory "")
+			(outputdirectory "../../Build/Aug 20 2026/")
 		)
 	)
@@
 		(descr "Keystone THM Miniature Test Point 5000-5004, http://www.keyelco.com/product-pdf.cfm?p=1309")
 		(tags "Through Hole Mount Test Points")
-		(property "Reference" "TP7"
+		(property "Reference" "TP1"
 			(at 0 -2.5 0)
 			(layer "F.SilkS")
@@
 		(descr "Keystone THM Miniature Test Point 5000-5004, http://www.keyelco.com/product-pdf.cfm?p=1309")
 		(tags "Through Hole Mount Test Points")
-		(property "Reference" "TP6"
+		(property "Reference" "TP5"
 			(at 0 -2.5 0)
 			(layer "F.SilkS")
@@
 		(descr "Keystone THM Miniature Test Point 5000-5004, http://www.keyelco.com/product-pdf.cfm?p=1309")
 		(tags "Through Hole Mount Test Points")
-		(property "Reference" "TP5"
+		(property "Reference" "TP4"
 			(at 0 -2.5 0)
 			(layer "F.SilkS")
@@
 		(descr "Keystone THM Miniature Test Point 5000-5004, http://www.keyelco.com/product-pdf.cfm?p=1309")
 		(tags "Through Hole Mount Test Points")
-		(property "Reference" "TP1"
+		(property "Reference" "TP2"
 			(at 0 -2.5 0)
 			(layer "F.SilkS")
@@
 		(descr "Keystone THM Miniature Test Point 5000-5004, http://www.keyelco.com/product-pdf.cfm?p=1309")
 		(tags "Through Hole Mount Test Points")
-		(property "Reference" "TP4"
+		(property "Reference" "TP3"
 			(at 0 -2.5 0)
 			(layer "F.SilkS")

Commit message: made all components THT on the buttons board
Parts:
- R1, R2, R3: footprint Resistor_SMD:R_0805_2012Metric -> Resistor_THT:R_Axial_DIN0207_L6.3mm_D2.5mm_P7.62mm_Horizontal
- moved R1 3.46 mm to (85.2, 69.0)
- moved R2 3.46 mm to (85.2, 86.5)
- moved R3 3.46 mm to (85.2, 104.0)
Routing:
- net GND: track 6.26 -> 0.00 mm, vias 3 -> 0
- net /Out3: track 36.0 -> 37.4 mm
- net /Out 1: track 63.6 -> 65.0 mm
- net /Out 2: track 49.8 -> 51.2 mm
